File: hdmi_lvds_converter.sch (EAGLE design)
At the start: 3 parts, among them J602 SS-53000-001, U1 DS90C387VJD/NOPB, U2 TFP401APZP

Commit message: - Change HDMI connector for better layout. - Start routing rgb signals.
Parts:
- J602: value SS-53000-001 -> 1759548-2; device ND_main_control_unit:SS-53000-001 -> ND_main_control_unit:1759548-2
Connections:
- new net E_B0: U1.B20, U2.QE0
- new net E_B1: U1.B21, U2.QE1
- new net E_B2: U1.B22, U2.QE2
- new net E_B3: U1.B23, U2.QE3
- new net E_B4: U1.B24, U2.QE4
- new net E_B5: U1.B25, U2.QE5
- new net E_B6: U1.B26, U2.QE6
- new net E_B7: U1.B27, U2.QE7
- new net E_G0: U1.G20, U2.QE8
- new net E_G1: U1.G21, U2.QE9
- new net E_G2: U1.G22, U2.QE10
- new net E_G3: U1.G23, U2.QE11
- new net E_G4: U1.G24, U2.QE12
- new net E_G5: U1.G25, U2.QE13
- new net E_G6: U1.G26, U2.QE14
- new net E_G7: U1.G27, U2.QE15
- new net E_R0: U1.R20, U2.QE16
- new net E_R1: U1.R21, U2.QE17
- new net E_R2: U1.R22, U2.QE18
- new net E_R3: U1.R23, U2.QE19
- new net E_R4: U1.R24, U2.QE20
- new net E_R5: U1.R25, U2.QE21
- new net E_R6: U1.R26, U2.QE22
- new net E_R7: U1.R27, U2.QE23
- new net N$25: U2.QO23
- new net N$26: U2.QO22
- new net N$27: U2.QO21
- new net N$28: U2.QO20
- new net N$29: U2.QO19
- new net N$30: U2.QO18
- new net N$31: U2.QO17
- new net N$32: U2.QO16
- new net N$33: U2.QO15
- new net N$34: U2.QO14
- new net N$35: U2.QO13
- new net N$36: U2.QO12
- new net N$37: U2.QO11
- new net N$38: U2.QO10
- new net N$39: U2.QO9
- new net N$40: U2.QO8
- new net N$41: U2.QO7
- new net N$42: U2.QO6
- new net N$43: U2.QO5
- new net N$44: U2.QO4
- new net N$45: U2.QO3
- new net N$46: U2.QO2
- new net N$47: U2.QO1
- new net N$48: U2.QO0
- new net N$57: U1.VSYNC
- new net N$58: U1.HSYNC
- new net N$59: U1.DUAL
- new net N$60: U1.DE
- new net N$61: U1.BAL
- new net N$62: U1.CLKIN
- new net O_B0: U1.B10
- new net O_B1: U1.B11
- new net O_B2: U1.B12
- new net O_B3: U1.B13
- new net O_B4: U1.B14
- new net O_B5: U1.B15
- new net O_B6: U1.B16
- new net O_B7: U1.B17
- new net O_G0: U1.G10
- new net O_G1: U1.G11
- new net O_G2: U1.G12
- new net O_G3: U1.G13
- new net O_G4: U1.G14
- new net O_G5: U1.G15
- new net O_G6: U1.G16
- new net O_G7: U1.G17
- new net O_R0: U1.R10
- new net O_R1: U1.R11
- new net O_R2: U1.R12
- new net O_R3: U1.R13
- new net O_R4: U1.R14
- new net O_R5: U1.R15
- new net O_R6: U1.R16
- new net O_R7: U1.R17
- net HDMI_CK_N: now also U2.RXC-
- net HDMI_CK_P: now also U2.RXC+
- net HDMI_D0_N: now also U2.RX0-
- net HDMI_D0_P: now also U2.RX0+
- net HDMI_D1_N: now also U2.RX1-
- net HDMI_D1_P: now also U2.RX1+
- net HDMI_D2_N: now also U2.RX2-
- net HDMI_D2_P: now also U2.RX2+

Commit message: - Latest changes
Connections:
- removed net N$25: U2.QO23
- removed net N$26: U2.QO22
- removed net N$27: U2.QO21
- removed net N$28: U2.QO20
- removed net N$29: U2.QO19
- removed net N$30: U2.QO18
- removed net N$31: U2.QO17
- removed net N$32: U2.QO16
- removed net N$33: U2.QO15
- removed net N$34: U2.QO14
- removed net N$35: U2.QO13
- removed net N$36: U2.QO12
- removed net N$37: U2.QO11
- removed net N$38: U2.QO10
- removed net N$39: U2.QO9
- removed net N$40: U2.QO8
- removed net N$41: U2.QO7
- removed net N$42: U2.QO6
- removed net N$43: U2.QO5
- removed net N$44: U2.QO4
- removed net N$45: U2.QO3
- removed net N$46: U2.QO2
- removed net N$47: U2.QO1
- removed net N$48: U2.QO0
- net O_B0: now also U2.QO0
- net O_B1: now also U2.QO1
- net O_B2: now also U2.QO2
- net O_B3: now also U2.QO3
- net O_B4: now also U2.QO4
- net O_B5: now also U2.QO5
- net O_B6: now also U2.QO6
- net O_B7: now also U2.QO7
- net O_G0: now also U2.QO8
- net O_G1: now also U2.QO9
- net O_G2: now also U2.QO10
- net O_G3: now also U2.QO11
- net O_G4: now also U2.QO12
- net O_G5: now also U2.QO13
- net O_G6: now also U2.QO14
- net O_G7: now also U2.QO15
- net O_R0: now also U2.QO16
- net O_R1: now also U2.QO17
- net O_R2: now also U2.QO18
- net O_R3: now also U2.QO19
- net O_R4: now also U2.QO20
- net O_R5: now also U2.QO21
- net O_R6: now also U2.QO22
- net O_R7: now also U2.QO23
